Commit message: control launch files work now

File: apple_description/urdf/apple.gazebo.xacro (robot description, xacro)
@@ -2,11 +2,5 @@
 <robot name="apple" xmlns:xacro="http://www.ros.org/wiki/xacro">
   <xacro:macro name="apple_gazebo" params="name">
-    <!-- ros_control plugin -->
-   <!-- <gazebo>
-      <plugin name="gazebo_ros_control" filename="libgazebo_ros_control.so">
-	<robotNamespace>/velvet_fingers</robotNamespace>
-      </plugin>
-    </gazebo> -->
-    <!-- Palm -->
+    <!-- Dummy Citi Truck base -->
     <gazebo reference="${name}_base">
       <material>Gazebo/White</material>

File: apple_description/urdf/apple.urdf.xacro (robot description, xacro)
@@ -9,9 +9,11 @@
   <!--Include a dummy CitiTruck for now-->
   <xacro:include filename="$(find apple_description)/urdf/dummy_citi_truck.xacro"/>
+ <!-- Gazebo plugins -->
+  <xacro:include filename="$(find apple_description)/gazebo/gazebo.urdf.xacro"/>
   <!-- Fix to world just for testing -->
   <link name="world"/>
   <!-- dummy citi truck-->
   <xacro:dummy_citi_truck name="dummy_citi_truck" parent="world">
-    <origin xyz="0 0 0" rpy="0 0 0" />
+    <origin xyz="0 0 0.15" rpy="0 0 0" />
   </xacro:dummy_citi_truck>
   <!--lbr -->
