Commit message: hqp_controllers modified

File: apple_description/urdf/apple.urdf.xacro (robot description, xacro)
@@ -15,5 +15,5 @@
   <!-- dummy citi truck-->
   <xacro:dummy_citi_truck name="dummy_citi_truck" parent="world">
-    <origin xyz="0 0 0.15" rpy="0 0 0" />
+    <origin xyz="0 0 0" rpy="0 0 0" />
   </xacro:dummy_citi_truck>
   <!--lbr -->

Commit message: apple_description: changed citi truck cad file and updated geometry

File: apple_description/urdf/apple.urdf.xacro (robot description, xacro)
@@ -7,21 +7,27 @@
   <!--Include the Velvet Fingers gripper-->
   <xacro:include filename="$(find velvet_fingers_description)/urdf/velvet_fingers.xacro"/>
-  <!--Include a dummy CitiTruck for now-->
-  <xacro:include filename="$(find apple_description)/urdf/dummy_citi_truck.xacro"/>
+   <!--Include the CitiTruck-->
+  <xacro:include filename="$(find apple_description)/urdf/citi_truck.xacro"/>
+  <!--Include the dummy CitiTruck (simplified geometry)-->
+  <!--xacro:include filename="$(find apple_description)/urdf/dummy_citi_truck.xacro"/-->
  <!-- Gazebo plugins -->
   <xacro:include filename="$(find apple_description)/gazebo/gazebo.urdf.xacro"/>
   <!-- Fix to world just for testing -->
   <link name="world"/>
+  <!-- citi truck-->
+  <xacro:citi_truck name="citi_truck" parent="world">
+    <origin xyz="0 0 0" rpy="0 0 0" />
+  </xacro:citi_truck>
   <!-- dummy citi truck-->
-  <xacro:dummy_citi_truck name="dummy_citi_truck" parent="world">
+  <!--xacro:dummy_citi_truck name="dummy_citi_truck" parent="world">
     <origin xyz="0 0 0" rpy="0 0 0" />
-  </xacro:dummy_citi_truck>
+  </xacro:dummy_citi_truck-->
   <!--lbr -->
-  <xacro:lbr_iiwa name="lbr_iiwa" hardware_interface="$(arg prefix)" parent="dummy_citi_truck_base">
-    <origin xyz="0.1 -0.2 0.45" rpy="0 ${PI / 2} ${-PI / 4}" />
+  <xacro:lbr_iiwa name="lbr_iiwa" hardware_interface="$(arg prefix)" parent="citi_truck_base">
+    <origin xyz="0.114 -0.265 0.5" rpy="0 ${PI / 2} ${-PI / 4}" />
   </xacro:lbr_iiwa>
   <!--velvet fingers gripper -->
   <xacro:velvet_fingers name="velvet_fingers" hardware_interface="$(arg prefix)" parent="lbr_iiwa_link_7">
-    <origin xyz="0 0 0.045" rpy="0 ${-PI / 2} 0" />
+    <origin xyz="0 0 0.065" rpy="0 ${-PI / 2} 0" />
   </xacro:velvet_fingers>
 </robot>

Commit message: added hqp_controllers_msgs package

File: apple_description/urdf/apple.urdf.xacro (robot description, xacro)
@@ -9,6 +9,4 @@
    <!--Include the CitiTruck-->
   <xacro:include filename="$(find apple_description)/urdf/citi_truck.xacro"/>
-  <!--Include the dummy CitiTruck (simplified geometry)-->
-  <!--xacro:include filename="$(find apple_description)/urdf/dummy_citi_truck.xacro"/-->
  <!-- Gazebo plugins -->
   <xacro:include filename="$(find apple_description)/gazebo/gazebo.urdf.xacro"/>
@@ -19,8 +17,4 @@
     <origin xyz="0 0 0" rpy="0 0 0" />
   </xacro:citi_truck>
-  <!-- dummy citi truck-->
-  <!--xacro:dummy_citi_truck name="dummy_citi_truck" parent="world">
-    <origin xyz="0 0 0" rpy="0 0 0" />
-  </xacro:dummy_citi_truck-->
   <!--lbr -->
   <xacro:lbr_iiwa name="lbr_iiwa" hardware_interface="$(arg prefix)" parent="citi_truck_base">

Commit message: apple_description: fixed intersecting citi_truck urdf file which messed up the controllers

File: apple_description/urdf/apple.urdf.xacro (robot description, xacro)
@@ -15,5 +15,5 @@
   <!-- citi truck-->
   <xacro:citi_truck name="citi_truck" parent="world">
-    <origin xyz="0 0 0" rpy="0 0 0" />
+    <origin xyz="0 0 0.2" rpy="0 0 0" />
   </xacro:citi_truck>
   <!--lbr -->

Commit message: added demo_palletizing node

File: apple_description/urdf/apple.urdf.xacro (robot description, xacro)
@@ -9,4 +9,6 @@
    <!--Include the CitiTruck-->
   <xacro:include filename="$(find apple_description)/urdf/citi_truck.xacro"/>
+   <!--Include the half pallet-->
+  <xacro:include filename="$(find apple_description)/urdf/half_pallet.xacro"/>
  <!-- Gazebo plugins -->
   <xacro:include filename="$(find apple_description)/gazebo/gazebo.urdf.xacro"/>
@@ -15,6 +17,14 @@
   <!-- citi truck-->
   <xacro:citi_truck name="citi_truck" parent="world">
-    <origin xyz="0 0 0.2" rpy="0 0 0" />
+    <origin xyz="0 0 0.15" rpy="0 0 0" />
   </xacro:citi_truck>
+  <!-- half pallet on the citi truck-->
+  <xacro:half_pallet name="transport_pallet" parent="citi_truck_base">
+    <origin xyz="0.52 0 -0.109" rpy="0 0 0" />
+  </xacro:half_pallet>
+  <!-- half pallet for loading -->
+  <xacro:half_pallet name="load_pallet" parent="world">
+    <origin xyz="0.52 -0.84 0.001" rpy="0 0 0" />
+  </xacro:half_pallet>
   <!--lbr -->
   <xacro:lbr_iiwa name="lbr_iiwa" hardware_interface="$(arg prefix)" parent="citi_truck_base">

File: apple_description/urdf/half_pallet.xacro (robot description, xacro)
@@ -5,6 +5,6 @@
   <!-- Import all Gazebo-customization elements, including Gazebo colors -->
   <xacro:include filename="$(find apple_description)/urdf/apple.gazebo.xacro" />
-  <xacro:macro name="citi_truck" params="parent name *origin">
-    <!--joint between {parent} and City Truck base -->
+  <xacro:macro name="half_pallet" params="parent name *origin">
+    <!--joint between {parent} and half_pallet -->
     <joint name="${parent}_${name}_joint" type="fixed">
       <insert_block name="origin"/>
@@ -14,21 +14,21 @@
     <link name="${name}_base">
       <inertial>
-        <origin xyz="-0.11 0.0 .31" rpy="0 0 0"/>
-        <mass value="30"/>
-        <inertia ixx="5"  ixy="0"  ixz="0" iyy="6" iyz="0" izz="2" />
+        <origin xyz="0.0 0.0 0.0" rpy="0 0 0"/>
+        <mass value="5.3"/>
+        <inertia ixx="0.48"  ixy="0"  ixz="0" iyy="0.25" iyz="0" izz="0.63" />
       </inertial>
       <visual>
         <origin xyz="0 0 0" rpy="0 0 0"/>
         <geometry>
-          <mesh filename="package://apple_description/meshes/citi_truck.stl"/>
+          <mesh filename="package://apple_description/meshes/half_pallet.stl"/>
         </geometry>
-        <material name="Aluminium"/>
+        <material name="Wood"/>
       </visual>
       <collision>
         <origin xyz="0 0 0" rpy="0 0 0"/>
         <geometry>
-          <mesh filename="package://apple_description/meshes/citi_truck.stl"/>
+          <mesh filename="package://apple_description/meshes/half_pallet.stl"/>
         </geometry>
-        <material name="Aluminium"/>
+        <material name="Wood"/>
       </collision>
     </link>

File: apple_description/urdf/materials.xacro (robot description, xacro)
@@ -28,3 +28,6 @@
     <color rgba="${118/255} ${115/255} ${111/255} 1.0"/>
   </material>
+  <material name="Wood">
+    <color rgba="${128/255} ${70/255} ${27/255} 1.0"/>
+  </material>
 </robot>

Commit message: demo_palletizing: apart from the task error monitoring, the demo works up to the grasp approach

File: apple_description/urdf/apple.urdf.xacro (robot description, xacro)
@@ -25,5 +25,5 @@
   <!-- half pallet for loading -->
   <xacro:half_pallet name="load_pallet" parent="world">
-    <origin xyz="0.52 -0.84 0.001" rpy="0 0 0" />
+    <origin xyz="0.8 -0.84 0.001" rpy="0 0 0" />
   </xacro:half_pallet>
   <!--lbr -->

Commit message: apple_description: changed apple urdf to account for the battery mounting

File: apple_description/urdf/apple.urdf.xacro (robot description, xacro)
@@ -21,5 +21,5 @@
   <!-- half pallet on the citi truck-->
   <xacro:half_pallet name="transport_pallet" parent="citi_truck_base">
-    <origin xyz="0.52 0 -0.109" rpy="0 0 0" />
+    <origin xyz="0.6 0 -0.109" rpy="0 0 0" />
   </xacro:half_pallet>
   <!-- half pallet for loading -->

Commit message: demo_palletizing: some demo tweaks

File: apple_description/urdf/apple.urdf.xacro (robot description, xacro)
@@ -25,5 +25,5 @@
   <!-- half pallet for loading -->
   <xacro:half_pallet name="load_pallet" parent="world">
-    <origin xyz="0.8 -0.84 0.001" rpy="0 0 0" />
+    <origin xyz="1.1 -0.9 0.001" rpy="0 0 0" />
   </xacro:half_pallet>
   <!--lbr -->

Commit message: aaand some more demo tweaks ...

File: apple_description/urdf/apple.urdf.xacro (robot description, xacro)
@@ -17,9 +17,9 @@
   <!-- citi truck-->
   <xacro:citi_truck name="citi_truck" parent="world">
-    <origin xyz="0 0 0.15" rpy="0 0 0" />
+    <origin xyz="0 0 0.09" rpy="0 0 0" />
   </xacro:citi_truck>
   <!-- half pallet on the citi truck-->
   <xacro:half_pallet name="transport_pallet" parent="citi_truck_base">
-    <origin xyz="0.6 0 -0.109" rpy="0 0 0" />
+    <origin xyz="0.6 0 -0.0899" rpy="0 0 0" />
   </xacro:half_pallet>
   <!-- half pallet for loading -->

Commit message: demo palletizing node flies again

File: apple_description/urdf/apple.urdf.xacro (robot description, xacro)
@@ -25,5 +25,5 @@
   <!-- half pallet for loading -->
   <xacro:half_pallet name="load_pallet" parent="world">
-    <origin xyz="1.1 -0.9 0.001" rpy="0 0 0" />
+    <origin xyz="1.1 -0.9 0.01" rpy="0 0 0" />
   </xacro:half_pallet>
   <!--lbr -->

Commit message: tweaked apple urdf

File: apple_description/urdf/apple.urdf.xacro (robot description, xacro)
@@ -21,5 +21,5 @@
   <!-- half pallet on the citi truck-->
   <xacro:half_pallet name="transport_pallet" parent="citi_truck_base">
-    <origin xyz="0.6 0 -0.0899" rpy="0 0 0" />
+    <origin xyz="0.6 0 -0.0699" rpy="0 0 0" />
   </xacro:half_pallet>
   <!-- half pallet for loading -->

Commit message: replaced world link with citi_truck_base

File: apple_description/urdf/apple.urdf.xacro (robot description, xacro)
@@ -17,17 +17,17 @@
   <!-- citi truck-->
   <xacro:citi_truck name="citi_truck" parent="world">
-    <origin xyz="0 0 0.09" rpy="0 0 0" />
+    <origin xyz="0 0 0" rpy="0 0 0" />
   </xacro:citi_truck>
   <!-- half pallet on the citi truck-->
   <xacro:half_pallet name="transport_pallet" parent="citi_truck_base">
-    <origin xyz="0.6 0 -0.0699" rpy="0 0 0" />
+    <origin xyz="0.6 0 0.02" rpy="0 0 0" />
   </xacro:half_pallet>
   <!-- half pallet for loading -->
-  <xacro:half_pallet name="load_pallet" parent="world">
+  <xacro:half_pallet name="load_pallet" parent="citi_truck_base">
     <origin xyz="1.1 -0.9 0.01" rpy="0 0 0" />
   </xacro:half_pallet>
   <!--lbr -->
   <xacro:lbr_iiwa name="lbr_iiwa" hardware_interface="$(arg prefix)" parent="citi_truck_base">
-    <origin xyz="0.114 -0.265 0.5" rpy="0 ${PI / 2} ${-PI / 4}" />
+    <origin xyz="0.114 -0.265 0.595" rpy="0 ${PI / 2} ${-PI / 4}" />
   </xacro:lbr_iiwa>
   <!--velvet fingers gripper -->

Commit message: modified the demo to the KUKA setting and added sphere beer avoidance

File: apple_description/urdf/apple.urdf.xacro (robot description, xacro)
@@ -25,5 +25,5 @@
   <!-- half pallet for loading -->
   <xacro:half_pallet name="load_pallet" parent="citi_truck_base">
-    <origin xyz="1.1 -0.9 0.01" rpy="0 0 0" />
+    <origin xyz="1.1 -0.9 0.02" rpy="0 0 0" />
   </xacro:half_pallet>
   <!--lbr -->
